File: Schematic/BoeBot-Schematic.sch (EAGLE design)
At the start: 53 parts, among them T1 FDN340P, U1 NCP1117ST50T3G, U2 LP2985-33DBVR, U3 ATMEGA16U2-MU(R), U5 LMV358IDGKR, X1 POWERSUPPLY_DC21MMX, X2 USB-B_TH, Y1 16MHz, Y2 CSTCE16M0V53-R0 16MHZ

Commit message: Added Servo's to Schematic
Parts:
- added U$2, U$3: IR_LED, Servo:IR_LED
Connections:
- net GND: now also U$2.GND, U$3.GND
- net MISO: now also U$3.CONTROL
- net SCK: now also U$2.CONTROL
Changed lines of the file:
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@@
 <layer number="54" name="bGND_GNDA" color="7" fill="1" visible="no" active="no"/>
 <layer number="56" name="wert" color="7" fill="1" visible="no" active="no"/>
+<layer number="90" name="Modules" color="5" fill="1" visible="yes" active="yes"/>
 <layer number="91" name="Nets" color="2" fill="1" visible="yes" active="yes"/>
 <layer number="92" name="Busses" color="1" fill="1" visible="yes" active="yes"/>
@@
 <part name="Y1" library="SmartPrj" deviceset="XTAL/S" device="" value="16MHz"/>
 <part name="U$1" library="SmartPrj" deviceset="DISCLAIMER" device=""/>
+<part name="U$2" library="Servo" deviceset="IR_LED" device=""/>
+<part name="U$3" library="Servo" deviceset="IR_LED" device=""/>
+<part name="GND6" library="supply1" deviceset="GND" device=""/>
+<part name="GND24" library="supply1" deviceset="GND" device=""/>
 </parts>
 <sheets>
@@
 <text x="226.06" y="96.52" size="1.778" layer="91">SCL</text>
 <text x="-83.82" y="-50.8" size="5.08" layer="91">Use of the ARDUINO name must be compliant with http://www.arduino.cc/en/Main/Policy</text>
-<wire x1="-116.84" y1="198.12" x2="-116.84" y2="195.58" width="2.54" layer="94"/>
-<wire x1="-116.84" y1="195.58" x2="-116.84" y2="5.08" width="2.54" layer="94"/>
+<wire x1="-116.84" y1="208.28" x2="-116.84" y2="5.08" width="2.54" layer="94"/>
 <wire x1="-116.84" y1="5.08" x2="274.32" y2="5.08" width="2.54" layer="94"/>
 <wire x1="274.32" y1="5.08" x2="274.32" y2="208.28" width="2.54" layer="94"/>
 <wire x1="274.32" y1="208.28" x2="-116.84" y2="208.28" width="2.54" layer="94"/>
-<wire x1="-116.84" y1="208.28" x2="-116.84" y2="198.12" width="2.54" layer="94"/>
 </plain>
 <instances>
@@
 <instance part="Y1" gate="G$1" x="2.54" y="73.66" rot="R270"/>
 <instance part="U$1" gate="G$1" x="-83.82" y="-43.18"/>
+<instance part="U$2" gate="G$1" x="398.78" y="152.4"/>
+<instance part="U$3" gate="G$1" x="401.862759375" y="53.298553125"/>
+<instance part="GND6" gate="1" x="365.76" y="27.94"/>
+<instance part="GND24" gate="1" x="363.22" y="124.46"/>
 </instances>
 <busses>
@@
 <pinref part="RN2" gate="D" pin="2"/>
 <pinref part="GND15" gate="1" pin="GND"/>
+</segment>
+<segment>
+<pinref part="U$3" gate="G$1" pin="GND"/>
+<pinref part="GND6" gate="1" pin="GND"/>
+<wire x1="381.542759375" y1="45.678553125" x2="365.76" y2="45.678553125" width="0.1524" layer="91"/>
+<wire x1="365.76" y1="45.678553125" x2="365.76" y2="30.48" width="0.1524" layer="91"/>
+</segment>
+<segment>
+<pinref part="U$2" gate="G$1" pin="GND"/>
+<pinref part="GND24" gate="1" pin="GND"/>
+<wire x1="378.46" y1="144.78" x2="363.22" y2="144.78" width="0.1524" layer="91"/>
+<wire x1="363.22" y1="144.78" x2="363.22" y2="127" width="0.1524" layer="91"/>
 </segment>
 </net>
@@
 <pinref part="ICSP" gate="A" pin="3"/>
 <pinref part="ZU4" gate="G$1" pin="(SCK)PB5"/>
+<wire x1="220.98" y1="86.36" x2="342.9" y2="86.36" width="0.1524" layer="91"/>
+<wire x1="342.9" y1="86.36" x2="342.9" y2="160.02" width="0.1524" layer="91"/>
+<junction x="220.98" y="86.36"/>
+<pinref part="U$2" gate="G$1" pin="CONTROL"/>
+<wire x1="342.9" y1="160.02" x2="378.46" y2="160.02" width="0.1524" layer="91"/>
 </segment>
 <segment>
@@
 <pinref part="ZU4" gate="G$1" pin="(MISO)PB4"/>
 <pinref part="IOH" gate="A" pin="5"/>
-<wire x1="220.98" y1="83.82" x2="251.46" y2="83.82" width="0.1524" layer="91"/>
+<pinref part="U$3" gate="G$1" pin="CONTROL"/>
+<wire x1="381.542759375" y1="60.918553125" x2="342.9" y2="60.918553125" width="0.1524" layer="91"/>
+<wire x1="342.9" y1="60.918553125" x2="342.9" y2="83.82" width="0.1524" layer="91"/>
+<wire x1="342.9" y1="83.82" x2="220.98" y2="83.82" width="0.1524" layer="91"/>
 <junction x="220.98" y="83.82"/>
 </segment>
