File: Schematic/BoeBot-Schematic.sch (EAGLE design)
At the start: 55 parts, among them T1 FDN340P, U1 NCP1117ST50T3G, U2 LP2985-33DBVR, U3 ATMEGA16U2-MU(R), U5 LMV358IDGKR, X1 POWERSUPPLY_DC21MMX, X2 USB-B_TH, Y1 16MHz, Y2 CSTCE16M0V53-R0 16MHZ

Commit message: Added IR_SENSORS to Schematic
Parts:
- added U$4, U$5: IR_SENSOR, IR_SENSOR:IR_SENSOR
Connections:
- net IO2 renamed N$4
- net +5V: now also U$4.VDD, U$5.VDD
- net GND: now also U$4.GND, U$5.GND
- net IO4: now also U$5.CONTROL
- net IO5: now also U$4.CONTROL
Changed lines of the file:
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@@
 <part name="P+12" library="supply1" deviceset="+5V" device=""/>
 <part name="P+13" library="supply1" deviceset="+5V" device=""/>
+<part name="U$4" library="IR_SENSOR" deviceset="IR_SENSOR" device=""/>
+<part name="U$5" library="IR_SENSOR" deviceset="IR_SENSOR" device=""/>
+<part name="P+14" library="supply1" deviceset="+5V" device=""/>
+<part name="P+15" library="supply1" deviceset="+5V" device=""/>
+<part name="GND25" library="supply1" deviceset="GND" device=""/>
+<part name="GND26" library="supply1" deviceset="GND" device=""/>
 </parts>
 <sheets>
@@
 <attribute name="VALUE" x="367.665" y="185.42" size="1.778" layer="96" rot="R180"/>
 </instance>
+<instance part="U$4" gate="G$1" x="485.14" y="137.16"/>
+<instance part="U$5" gate="G$1" x="485.14" y="78.74"/>
+<instance part="P+14" gate="1" x="459.74" y="96.52" smashed="yes">
+<attribute name="VALUE" x="461.645" y="99.06" size="1.778" layer="96" rot="R180"/>
+</instance>
+<instance part="P+15" gate="1" x="462.28" y="160.02" smashed="yes">
+<attribute name="VALUE" x="464.185" y="162.56" size="1.778" layer="96" rot="R180"/>
+</instance>
+<instance part="GND25" gate="1" x="462.28" y="116.84"/>
+<instance part="GND26" gate="1" x="459.74" y="58.42"/>
 </instances>
 <busses>
@@
 <wire x1="381.542759375" y1="53.34" x2="381.542759375" y2="53.298553125" width="0.1524" layer="91"/>
 </segment>
+<segment>
+<pinref part="P+15" gate="1" pin="+5V"/>
+<wire x1="462.28" y1="157.48" x2="462.28" y2="144.78" width="0.1524" layer="91"/>
+<pinref part="U$4" gate="G$1" pin="VDD"/>
+<wire x1="462.28" y1="144.78" x2="472.44" y2="144.78" width="0.1524" layer="91"/>
+</segment>
+<segment>
+<pinref part="P+14" gate="1" pin="+5V"/>
+<wire x1="459.74" y1="93.98" x2="459.74" y2="86.36" width="0.1524" layer="91"/>
+<pinref part="U$5" gate="G$1" pin="VDD"/>
+<wire x1="459.74" y1="86.36" x2="472.44" y2="86.36" width="0.1524" layer="91"/>
+</segment>
 </net>
 <net name="GND" class="2">
@@
 <wire x1="378.46" y1="144.78" x2="363.22" y2="144.78" width="0.1524" layer="91"/>
 <wire x1="363.22" y1="144.78" x2="363.22" y2="127" width="0.1524" layer="91"/>
+</segment>
+<segment>
+<pinref part="U$5" gate="G$1" pin="GND"/>
+<pinref part="GND26" gate="1" pin="GND"/>
+<wire x1="472.44" y1="78.74" x2="459.74" y2="78.74" width="0.1524" layer="91"/>
+<wire x1="459.74" y1="78.74" x2="459.74" y2="60.96" width="0.1524" layer="91"/>
+</segment>
+<segment>
+<pinref part="U$4" gate="G$1" pin="GND"/>
+<pinref part="GND25" gate="1" pin="GND"/>
+<wire x1="472.44" y1="137.16" x2="462.28" y2="137.16" width="0.1524" layer="91"/>
+<wire x1="462.28" y1="137.16" x2="462.28" y2="119.38" width="0.1524" layer="91"/>
 </segment>
 </net>
@@
 </segment>
 </net>
-<net name="IO2" class="0">
-<segment>
-<wire x1="220.98" y1="27.94" x2="200.66" y2="27.94" width="0.1524" layer="91"/>
-<wire x1="200.66" y1="27.94" x2="200.66" y2="30.48" width="0.1524" layer="91"/>
-<wire x1="200.66" y1="30.48" x2="175.26" y2="30.48" width="0.1524" layer="91"/>
-<label x="180.34" y="30.48" size="1.778" layer="95"/>
-<pinref part="IOL" gate="A" pin="3"/>
-<pinref part="ZU4" gate="G$1" pin="(INT0)PD2"/>
-</segment>
-</net>
 <net name="IO1" class="0">
 <segment>
@@
 <pinref part="IOL" gate="A" pin="5"/>
 <pinref part="ZU4" gate="G$1" pin="(T0)PD4"/>
+<pinref part="U$5" gate="G$1" pin="CONTROL"/>
+<wire x1="472.44" y1="71.12" x2="444.5" y2="71.12" width="0.1524" layer="91"/>
+<wire x1="444.5" y1="71.12" x2="444.5" y2="109.22" width="0.1524" layer="91"/>
+<wire x1="444.5" y1="109.22" x2="309.88" y2="109.22" width="0.1524" layer="91"/>
+<wire x1="309.88" y1="109.22" x2="309.88" y2="33.02" width="0.1524" layer="91"/>
+<wire x1="309.88" y1="33.02" x2="220.98" y2="33.02" width="0.1524" layer="91"/>
+<junction x="220.98" y="33.02"/>
 </segment>
 </net>
@@
 <pinref part="ZU4" gate="G$1" pin="(T1)PD5"/>
 <pinref part="IOL" gate="A" pin="6"/>
+<pinref part="U$4" gate="G$1" pin="CONTROL"/>
+<wire x1="472.44" y1="129.54" x2="444.5" y2="129.54" width="0.1524" layer="91"/>
+<wire x1="444.5" y1="129.54" x2="444.5" y2="111.76" width="0.1524" layer="91"/>
+<wire x1="444.5" y1="111.76" x2="307.34" y2="111.76" width="0.1524" layer="91"/>
+<wire x1="307.34" y1="111.76" x2="307.34" y2="35.56" width="0.1524" layer="91"/>
+<wire x1="220.98" y1="35.56" x2="307.34" y2="35.56" width="0.1524" layer="91"/>
+<junction x="220.98" y="35.56"/>
 </segment>
 </net>
@@
 </segment>
 </net>
+<net name="N$4" class="0">
+<segment>
+<pinref part="IOL" gate="A" pin="3"/>
+<wire x1="220.98" y1="27.94" x2="200.66" y2="27.94" width="0.1524" layer="91"/>
+<wire x1="200.66" y1="27.94" x2="200.66" y2="30.48" width="0.1524" layer="91"/>
+<wire x1="200.66" y1="30.48" x2="175.26" y2="30.48" width="0.1524" layer="91"/>
+<pinref part="ZU4" gate="G$1" pin="(INT0)PD2"/>
+<label x="180.34" y="30.48" size="1.778" layer="95"/>
+</segment>
+</net>

Commit message: Added IR_LED'S to Schematic
Parts:
- added R3, R4: (no value), resistor:R-US_0411/15
- added U$6, U$7: IR_LED, IR_LED:IR_LED
Connections:
- new net N$6: R3.1, U$6.CATHODE
- new net N$7: R4.1, U$7.CATHODE
- net IO6: now also U$6.ANODE
- net N$4: now also U$7.ANODE
Changed lines of the file:
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@@
 <layer number="97" name="Info" color="7" fill="1" visible="no" active="yes"/>
 <layer number="98" name="Guide" color="6" fill="1" visible="no" active="yes"/>
+<layer number="99" name="SpiceOrder" color="5" fill="1" visible="yes" active="yes"/>
 <layer number="100" name="Muster" color="7" fill="1" visible="no" active="yes"/>
 <layer number="101" name="Patch_Top" color="7" fill="1" visible="no" active="yes"/>
@@
 <part name="GND25" library="supply1" deviceset="GND" device=""/>
 <part name="GND26" library="supply1" deviceset="GND" device=""/>
+<part name="U$6" library="IR_LED" deviceset="IR_LED" device=""/>
+<part name="U$7" library="IR_LED" deviceset="IR_LED" device=""/>
+<part name="R3" library="resistor" deviceset="R-US_" device="0411/15"/>
+<part name="R4" library="resistor" deviceset="R-US_" device="0411/15"/>
 </parts>
 <sheets>
@@
 <instance part="GND25" gate="1" x="462.28" y="116.84"/>
 <instance part="GND26" gate="1" x="459.74" y="58.42"/>
+<instance part="U$6" gate="G$1" x="551.18" y="137.16" rot="R90"/>
+<instance part="U$7" gate="G$1" x="548.64" y="73.66" rot="R90"/>
+<instance part="R3" gate="G$1" x="604.52" y="137.16"/>
+<instance part="R4" gate="G$1" x="604.52" y="73.66"/>
 </instances>
 <busses>
@@
 <pinref part="U$5" gate="G$1" pin="CONTROL"/>
 <wire x1="472.44" y1="71.12" x2="444.5" y2="71.12" width="0.1524" layer="91"/>
-<wire x1="444.5" y1="71.12" x2="444.5" y2="109.22" width="0.1524" layer="91"/>
-<wire x1="444.5" y1="109.22" x2="309.88" y2="109.22" width="0.1524" layer="91"/>
-<wire x1="309.88" y1="109.22" x2="309.88" y2="33.02" width="0.1524" layer="91"/>
+<wire x1="444.5" y1="71.12" x2="444.5" y2="116.84" width="0.1524" layer="91"/>
+<wire x1="444.5" y1="116.84" x2="309.88" y2="116.84" width="0.1524" layer="91"/>
+<wire x1="309.88" y1="116.84" x2="309.88" y2="33.02" width="0.1524" layer="91"/>
 <wire x1="309.88" y1="33.02" x2="220.98" y2="33.02" width="0.1524" layer="91"/>
 <junction x="220.98" y="33.02"/>
@@
 <pinref part="U$4" gate="G$1" pin="CONTROL"/>
 <wire x1="472.44" y1="129.54" x2="444.5" y2="129.54" width="0.1524" layer="91"/>
-<wire x1="444.5" y1="129.54" x2="444.5" y2="111.76" width="0.1524" layer="91"/>
-<wire x1="444.5" y1="111.76" x2="307.34" y2="111.76" width="0.1524" layer="91"/>
-<wire x1="307.34" y1="111.76" x2="307.34" y2="35.56" width="0.1524" layer="91"/>
+<wire x1="444.5" y1="129.54" x2="444.5" y2="119.38" width="0.1524" layer="91"/>
+<wire x1="444.5" y1="119.38" x2="307.34" y2="119.38" width="0.1524" layer="91"/>
+<wire x1="307.34" y1="119.38" x2="307.34" y2="35.56" width="0.1524" layer="91"/>
 <wire x1="220.98" y1="35.56" x2="307.34" y2="35.56" width="0.1524" layer="91"/>
 <junction x="220.98" y="35.56"/>
@@
 <pinref part="IOL" gate="A" pin="7"/>
 <pinref part="ZU4" gate="G$1" pin="(AIN0)PD6"/>
+<pinref part="U$6" gate="G$1" pin="ANODE"/>
+<wire x1="530.86" y1="137.16" x2="518.16" y2="137.16" width="0.1524" layer="91"/>
+<wire x1="518.16" y1="137.16" x2="518.16" y2="104.14" width="0.1524" layer="91"/>
+<wire x1="518.16" y1="104.14" x2="332.74" y2="104.14" width="0.1524" layer="91"/>
+<wire x1="332.74" y1="104.14" x2="332.74" y2="38.1" width="0.1524" layer="91"/>
+<wire x1="332.74" y1="38.1" x2="220.98" y2="38.1" width="0.1524" layer="91"/>
+<junction x="220.98" y="38.1"/>
 </segment>
 </net>
@@
 <pinref part="ZU4" gate="G$1" pin="(INT0)PD2"/>
 <label x="180.34" y="30.48" size="1.778" layer="95"/>
-</segment>
-</net>
+<pinref part="U$7" gate="G$1" pin="ANODE"/>
+<wire x1="528.32" y1="73.66" x2="518.16" y2="73.66" width="0.1524" layer="91"/>
+<wire x1="518.16" y1="73.66" x2="518.16" y2="101.6" width="0.1524" layer="91"/>
+<wire x1="518.16" y1="101.6" x2="335.28" y2="101.6" width="0.1524" layer="91"/>
+<wire x1="335.28" y1="101.6" x2="335.28" y2="27.94" width="0.1524" layer="91"/>
+<wire x1="335.28" y1="27.94" x2="220.98" y2="27.94" width="0.1524" layer="91"/>
+<junction x="220.98" y="27.94"/>
+</segment>
+</net>
+<net name="N$6" class="0">
+<segment>
+<pinref part="U$6" gate="G$1" pin="CATHODE"/>
+<pinref part="R3" gate="G$1" pin="1"/>
+<wire x1="581.66" y1="137.16" x2="599.44" y2="137.16" width="0.1524" layer="91"/>
+</segment>
+</net>
+<net name="N$7" class="0">
+<segment>
+<pinref part="U$7" gate="G$1" pin="CATHODE"/>
+<pinref part="R4" gate="G$1" pin="1"/>
+<wire x1="579.12" y1="73.66" x2="599.44" y2="73.66" width="0.1524" layer="91"/>
+</segment>
+</net>

Commit message: Completed Schematic
Parts:
- added R5, R6: 220R, resistor:R-US_0207/2V
- added R7: 1k, resistor:R-US_0207/2V
- added RIGHT_IR_LED: asdfa, IR_SENSOR:IR_SENSOR
- added RIGHT_SERVO: IR_LED, Servo:IR_LED
- R3, R4: value (none) -> 12K
- U$2: value IR_LED -> BUZZER; device Servo:IR_LED -> BUZZER:BUZZER
- U$4: value IR_SENSOR -> IR_LED; device IR_SENSOR:IR_SENSOR -> IR_LED:IR_LED
Connections:
- new net N$2: R4.2, U$7.ANODE
- new net N$5: R3.2, U$6.ANODE
- new net N$8: R7.2, U$4.ANODE
- new net N$9: ICSP.3, IOH.6, RIGHT_SERVO.CONTROL, ZU4.(SCK)PB5
- net +5V: now also RIGHT_IR_LED.VDD, RIGHT_SERVO.VDD; no longer U$2.VDD, U$4.VDD
- net GND: now also RIGHT_IR_LED.GND, RIGHT_SERVO.GND, U$2.CATHODE, U$4.CATHODE, U$6.CATHODE, U$7.CATHODE; no longer U$2.GND, U$4.GND
- net IO4: now also R6.1; no longer U$5.CONTROL
- net IO5: now also R5.1; no longer U$4.CONTROL
- net IO6: now also R3.1; no longer U$6.ANODE
- net IO7: now also R7.1
- net N$4: now also R4.1; no longer U$7.ANODE
- net N$6: now also R5.2, RIGHT_IR_LED.CONTROL; no longer R3.1, U$6.CATHODE
- net N$7: now also R6.2, U$5.CONTROL; no longer R4.1, U$7.CATHODE
- net SCK: no longer ICSP.3, IOH.6, U$2.CONTROL, ZU4.(SCK)PB5
- net SS: now also U$2.ANODE
Other:
- note added: "BUZZER"
- note added: "FONT_IR_LED"
- note added: "FRONT_IR_SENSOR"
- note added: "LEFT SERVO"
- note added: "RED_LED"
- note added: "RIGHT SERVO"
- note added: "RIGHT_IR_LED"
- note added: "RIGHT_IR_SENSOR"
- moved on the sheet: R3, R4

Commit message: Added a Description to the Schematic
Other:
- note added: "The Servo Motors, IR-Sensors, IR-LED's and the Buzzer were connected to the Parallax Shield and Arduino as indicated above. Resistor values were manipulated to obtain and optimal detection range. Common Problems: -The IR-Sensors and IR-LED's would keep getting out of alignment so the stopping distance would not be consistent. (A better solution would have been to use a single device rather than 2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"
Changed lines of the file:
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@@
 <wire x1="723.9" y1="5.08" x2="292.1" y2="5.08" width="2.54" layer="94"/>
 <wire x1="292.1" y1="5.08" x2="292.1" y2="210.82" width="2.54" layer="94"/>
+<text x="297.18" y="-55.88" size="5.08" layer="91">The Servo Motors, IR-Sensors, IR-LED's and the Buzzer were connected to the Parallax Shield and Arduino as indicated above.
+Resistor values were manipulated to obtain and optimal detection range.
+Common Problems:
+-The IR-Sensors and IR-LED's would keep getting out of alignment so the stopping distance would not be consistent.
+(A better solution would have been to use a single device rather than 2 seperate devices working together)
+</text>
 </plain>
 <instances>
@@
 </schematic>
 </drawing>
+<compatibility>
+<note version="6.3" minversion="6.2.2" severity="warning">
+Since Version 6.2.2 text objects can contain more than one line,
+which will not be processed correctly with this version.
+</note>
+</compatibility>
 </eagle>
